File: ch552_promicro.kicad_sch (KiCad schematic)
At the start: 9 parts, among them J1 Conn_01x12, J2 Conn_01x12, J3 USB_C_Receptacle_USB2.0, U1 CH552T

Commit message: Preparing a README.
Other:
- company: (none) -> Namnlos
- title: (none) -> CH552T ProMicro
Changed lines of the file:
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@@
 (kicad_sch (version 20230121) (generator eeschema)
   (paper "A4")
+  (title_block
+    (title "CH552T ProMicro")
+    (date "2023-10-21")
+    (rev "v0.1")
+    (company "Namnlos")
+    (comment 1 "Jan Lindblom")
+  )
   (junction (at 50.8 160.02) (diameter 0) (color 0 0 0 0)
   )
